Commit message: Add ISIMM ROS 2 robot package

File: ros2_ws/src/isimm_robot/urdf/robot.urdf.xacro (robot description, xacro)
@@ -1,24 +1,169 @@
-<!-- Dimensions robot -->
-<xacro:property name="robot_length" value="0.57"/>
-<xacro:property name="robot_width"  value="0.40"/>
-<xacro:property name="robot_total_height" value="0.30"/>
-<!-- Plateaux -->
-<xacro:property name="plate_thickness" value="0.01"/>
-<!-- Roues hoverboard -->
-<xacro:property name="wheel_diameter" value="0.165"/>
-<xacro:property name="wheel_radius" value="0.0825"/>
-<xacro:property name="wheel_width" value="0.08"/>
-<!-- Distance réelle entre centres des roues -->
-<xacro:property name="wheel_separation" value="0.48"/>
-<!-- Roues centrées longitudinalement -->
-<xacro:property name="wheel_x" value="0.0"/>
-<!-- LiDAR -->
-<xacro:property name="laser_height" value="0.24"/>
-<xacro:property name="laser_x" value="0.0"/>
-<xacro:property name="laser_y" value="0.0"/>
-<!-- IMU -->
-<xacro:property name="imu_x" value="0.0"/>
-<xacro:property name="imu_y" value="0.0"/>
-<xacro:property name="imu_z" value="0.29"/>
-<!-- Masse estimée -->
-<xacro:property name="body_mass" value="10.0"/>
+<?xml version="1.0"?>
+<robot name="isimm_robot" xmlns:xacro="http://www.ros.org/wiki/xacro">
+  <!-- Argument conservé pour compatibilité avec le launch file (robot.launch.py
+       le passe toujours à xacro). Aucun joint_state_publisher_gui n'est lancé
+       dans l'architecture actuelle (pas d'encodeurs, pas de ros2_control) :
+       cet argument n'a donc aucun effet fonctionnel pour l'instant. -->
+  <xacro:arg name="use_joint_state_gui" default="false"/>
+  <!-- ===================== Dimensions robot ===================== -->
+  <xacro:property name="robot_length" value="0.57"/>
+  <xacro:property name="robot_width"  value="0.40"/>
+  <xacro:property name="robot_total_height" value="0.30"/>
+  <!-- Plateaux -->
+  <xacro:property name="plate_thickness" value="0.01"/>
+  <!-- Roues hoverboard -->
+  <xacro:property name="wheel_diameter" value="0.165"/>
+  <xacro:property name="wheel_radius" value="0.0825"/>
+  <xacro:property name="wheel_width" value="0.08"/>
+  <!-- Distance réelle entre centres des roues (validée) -->
+  <xacro:property name="wheel_separation" value="0.48"/>
+  <!-- Roues centrées longitudinalement -->
+  <xacro:property name="wheel_x" value="0.0"/>
+  <!-- Roues au niveau du sol : centre roue = rayon roue au-dessus de base_footprint -->
+  <xacro:property name="wheel_z" value="${wheel_radius}"/>
+  <!-- base_link surélevé du rayon de roue par rapport à base_footprint -->
+  <xacro:property name="base_link_z" value="${wheel_radius}"/>
+  <!-- LiDAR (validé) -->
+  <xacro:property name="laser_height" value="0.24"/>
+  <xacro:property name="laser_x" value="0.0"/>
+  <xacro:property name="laser_y" value="0.0"/>
+  <xacro:property name="laser_radius" value="0.038"/>
+  <xacro:property name="laser_length" value="0.05"/>
+  <!-- IMU (validé) -->
+  <xacro:property name="imu_x" value="0.0"/>
+  <xacro:property name="imu_y" value="0.0"/>
+  <xacro:property name="imu_z" value="0.32"/>
+  <xacro:property name="imu_size" value="0.02"/>
+  <!-- Masse estimée -->
+  <xacro:property name="body_mass" value="10.0"/>
+  <xacro:property name="wheel_mass" value="1.0"/>
+  <!-- Couleurs -->
+  <material name="isimm_grey">
+    <color rgba="0.5 0.5 0.5 1.0"/>
+  </material>
+  <material name="isimm_black">
+    <color rgba="0.05 0.05 0.05 1.0"/>
+  </material>
+  <material name="isimm_red">
+    <color rgba="0.8 0.0 0.0 1.0"/>
+  </material>
+  <!-- ===================== Macro inertie boîte ===================== -->
+  <xacro:macro name="box_inertia" params="mass x y z">
+    <inertial>
+      <mass value="${mass}"/>
+      <inertia
+        ixx="${mass / 12.0 * (y*y + z*z)}" ixy="0.0" ixz="0.0"
+        iyy="${mass / 12.0 * (x*x + z*z)}" iyz="0.0"
+        izz="${mass / 12.0 * (x*x + y*y)}"/>
+    </inertial>
+  </xacro:macro>
+  <xacro:macro name="cylinder_inertia" params="mass r h">
+    <inertial>
+      <mass value="${mass}"/>
+      <inertia
+        ixx="${mass / 12.0 * (3*r*r + h*h)}" ixy="0.0" ixz="0.0"
+        iyy="${mass / 12.0 * (3*r*r + h*h)}" iyz="0.0"
+        izz="${mass * r*r / 2.0}"/>
+    </inertial>
+  </xacro:macro>
+  <!-- ===================== base_footprint ===================== -->
+  <!-- Frame virtuel, projeté au sol, sans géométrie. Référence pour Nav2/costmaps. -->
+  <link name="base_footprint"/>
+  <joint name="base_footprint_joint" type="fixed">
+    <parent link="base_footprint"/>
+    <child link="base_link"/>
+    <origin xyz="0 0 ${base_link_z}" rpy="0 0 0"/>
+  </joint>
+  <!-- ===================== base_link ===================== -->
+  <link name="base_link">
+    <visual>
+      <origin xyz="0 0 0" rpy="0 0 0"/>
+      <geometry>
+        <box size="${robot_length} ${robot_width} ${robot_total_height}"/>
+      </geometry>
+      <material name="isimm_grey"/>
+    </visual>
+    <collision>
+      <origin xyz="0 0 0" rpy="0 0 0"/>
+      <geometry>
+        <box size="${robot_length} ${robot_width} ${robot_total_height}"/>
+      </geometry>
+    </collision>
+    <xacro:box_inertia mass="${body_mass}" x="${robot_length}" y="${robot_width}" z="${robot_total_height}"/>
+  </link>
+  <!-- ===================== Roues ===================== -->
+  <!-- Pas d'encodeurs, pas de ros2_control : les roues sont donc modélisées
+       en joints fixes (pas d'état articulaire publié). L'odométrie réelle
+       vient de rf2o (recalage LiDAR), pas de la cinématique des roues. -->
+  <xacro:macro name="wheel" params="prefix reflect">
+    <link name="${prefix}_wheel_link">
+      <visual>
+        <origin xyz="0 0 0" rpy="${pi/2} 0 0"/>
+        <geometry>
+          <cylinder radius="${wheel_radius}" length="${wheel_width}"/>
+        </geometry>
+        <material name="isimm_black"/>
+      </visual>
+      <collision>
+        <origin xyz="0 0 0" rpy="${pi/2} 0 0"/>
+        <geometry>
+          <cylinder radius="${wheel_radius}" length="${wheel_width}"/>
+        </geometry>
+      </collision>
+      <xacro:cylinder_inertia mass="${wheel_mass}" r="${wheel_radius}" h="${wheel_width}"/>
+    </link>
+    <joint name="${prefix}_wheel_joint" type="fixed">
+      <parent link="base_link"/>
+      <child link="${prefix}_wheel_link"/>
+      <origin xyz="${wheel_x} ${reflect * wheel_separation / 2.0} ${-base_link_z + wheel_z}" rpy="0 0 0"/>
+    </joint>
+  </xacro:macro>
+  <xacro:wheel prefix="left" reflect="1"/>
+  <xacro:wheel prefix="right" reflect="-1"/>
+  <!-- ===================== LiDAR ===================== -->
+  <link name="laser_link">
+    <visual>
+      <origin xyz="0 0 0" rpy="0 0 0"/>
+      <geometry>
+        <cylinder radius="${laser_radius}" length="${laser_length}"/>
+      </geometry>
+      <material name="isimm_black"/>
+    </visual>
+    <collision>
+      <origin xyz="0 0 0" rpy="0 0 0"/>
+      <geometry>
+        <cylinder radius="${laser_radius}" length="${laser_length}"/>
+      </geometry>
+    </collision>
+    <xacro:cylinder_inertia mass="0.2" r="${laser_radius}" h="${laser_length}"/>
+  </link>
+  <joint name="laser_joint" type="fixed">
+    <parent link="base_link"/>
+    <child link="laser_link"/>
+    <!-- laser_height est donné depuis base_footprint (sol) -> on retire base_link_z -->
+    <origin xyz="${laser_x} ${laser_y} ${laser_height - base_link_z}" rpy="0 0 0"/>
+  </joint>
+  <!-- ===================== IMU ===================== -->
+  <link name="imu_link">
+    <visual>
+      <origin xyz="0 0 0" rpy="0 0 0"/>
+      <geometry>
+        <box size="${imu_size} ${imu_size} ${imu_size}"/>
+      </geometry>
+      <material name="isimm_red"/>
+    </visual>
+    <collision>
+      <origin xyz="0 0 0" rpy="0 0 0"/>
+      <geometry>
+        <box size="${imu_size} ${imu_size} ${imu_size}"/>
+      </geometry>
+    </collision>
+    <xacro:box_inertia mass="0.05" x="${imu_size}" y="${imu_size}" z="${imu_size}"/>
+  </link>
+  <joint name="imu_joint" type="fixed">
+    <parent link="base_link"/>
+    <child link="imu_link"/>
+    <!-- imu_z est donné depuis base_footprint (sol) -> on retire base_link_z -->
+    <origin xyz="${imu_x} ${imu_y} ${imu_z - base_link_z}" rpy="0 0 0"/>
+  </joint>
+</robot>

Commit message: Update ROS2 robot, navigation, SLAM and scripts

File: ros2_ws/src/isimm_robot/urdf/robot.urdf.xacro (robot description, xacro)
@@ -1,28 +1,18 @@
 <?xml version="1.0"?>
 <robot name="isimm_robot" xmlns:xacro="http://www.ros.org/wiki/xacro">
-  <!-- Argument conservé pour compatibilité avec le launch file (robot.launch.py
-       le passe toujours à xacro). Aucun joint_state_publisher_gui n'est lancé
-       dans l'architecture actuelle (pas d'encodeurs, pas de ros2_control) :
-       cet argument n'a donc aucun effet fonctionnel pour l'instant. -->
-  <xacro:arg name="use_joint_state_gui" default="false"/>
-  <!-- ===================== Dimensions robot ===================== -->
+  <!-- TF : base_link est la RACINE (odom -> base_link est publié par RF2O).
+       Pas de base_footprint : deux parents pour base_link casseraient TF. -->
+  <!-- Dimensions robot -->
   <xacro:property name="robot_length" value="0.57"/>
   <xacro:property name="robot_width"  value="0.40"/>
   <xacro:property name="robot_total_height" value="0.30"/>
-  <!-- Plateaux -->
-  <xacro:property name="plate_thickness" value="0.01"/>
   <!-- Roues hoverboard -->
-  <xacro:property name="wheel_diameter" value="0.165"/>
   <xacro:property name="wheel_radius" value="0.0825"/>
   <xacro:property name="wheel_width" value="0.08"/>
-  <!-- Distance réelle entre centres des roues (validée) -->
+  <!-- Entraxe réel validé (= wheel_separation du motor controller) -->
   <xacro:property name="wheel_separation" value="0.48"/>
-  <!-- Roues centrées longitudinalement -->
-  <xacro:property name="wheel_x" value="0.0"/>
-  <!-- Roues au niveau du sol : centre roue = rayon roue au-dessus de base_footprint -->
-  <xacro:property name="wheel_z" value="${wheel_radius}"/>
-  <!-- base_link surélevé du rayon de roue par rapport à base_footprint -->
+  <!-- base_link = centre de l'axe des roues, à wheel_radius du sol -->
   <xacro:property name="base_link_z" value="${wheel_radius}"/>
-  <!-- LiDAR (validé) -->
+  <!-- LiDAR (hauteur depuis le sol) -->
   <xacro:property name="laser_height" value="0.24"/>
   <xacro:property name="laser_x" value="0.0"/>
@@ -30,23 +20,14 @@
   <xacro:property name="laser_radius" value="0.038"/>
   <xacro:property name="laser_length" value="0.05"/>
-  <!-- IMU (validé) -->
+  <!-- IMU (hauteur depuis le sol) -->
   <xacro:property name="imu_x" value="0.0"/>
   <xacro:property name="imu_y" value="0.0"/>
   <xacro:property name="imu_z" value="0.32"/>
   <xacro:property name="imu_size" value="0.02"/>
-  <!-- Masse estimée -->
   <xacro:property name="body_mass" value="10.0"/>
   <xacro:property name="wheel_mass" value="1.0"/>
-  <!-- Couleurs -->
-  <material name="isimm_grey">
-    <color rgba="0.5 0.5 0.5 1.0"/>
-  </material>
-  <material name="isimm_black">
-    <color rgba="0.05 0.05 0.05 1.0"/>
-  </material>
-  <material name="isimm_red">
-    <color rgba="0.8 0.0 0.0 1.0"/>
-  </material>
-  <!-- ===================== Macro inertie boîte ===================== -->
+  <material name="isimm_grey"><color rgba="0.5 0.5 0.5 1.0"/></material>
+  <material name="isimm_black"><color rgba="0.05 0.05 0.05 1.0"/></material>
+  <material name="isimm_red"><color rgba="0.8 0.0 0.0 1.0"/></material>
   <xacro:macro name="box_inertia" params="mass x y z">
     <inertial>
@@ -67,47 +48,28 @@
     </inertial>
   </xacro:macro>
-  <!-- ===================== base_footprint ===================== -->
-  <!-- Frame virtuel, projeté au sol, sans géométrie. Référence pour Nav2/costmaps. -->
-  <link name="base_footprint"/>
-  <joint name="base_footprint_joint" type="fixed">
-    <parent link="base_footprint"/>
-    <child link="base_link"/>
-    <origin xyz="0 0 ${base_link_z}" rpy="0 0 0"/>
-  </joint>
-  <!-- ===================== base_link ===================== -->
+  <!-- ===================== base_link (racine) ===================== -->
   <link name="base_link">
     <visual>
-      <origin xyz="0 0 0" rpy="0 0 0"/>
-      <geometry>
-        <box size="${robot_length} ${robot_width} ${robot_total_height}"/>
-      </geometry>
+      <origin xyz="0 0 ${robot_total_height/2 - base_link_z + 0.02}" rpy="0 0 0"/>
+      <geometry><box size="${robot_length} ${robot_width} ${robot_total_height}"/></geometry>
       <material name="isimm_grey"/>
     </visual>
     <collision>
-      <origin xyz="0 0 0" rpy="0 0 0"/>
-      <geometry>
-        <box size="${robot_length} ${robot_width} ${robot_total_height}"/>
-      </geometry>
+      <origin xyz="0 0 ${robot_total_height/2 - base_link_z + 0.02}" rpy="0 0 0"/>
+      <geometry><box size="${robot_length} ${robot_width} ${robot_total_height}"/></geometry>
     </collision>
     <xacro:box_inertia mass="${body_mass}" x="${robot_length}" y="${robot_width}" z="${robot_total_height}"/>
   </link>
-  <!-- ===================== Roues ===================== -->
-  <!-- Pas d'encodeurs, pas de ros2_control : les roues sont donc modélisées
-       en joints fixes (pas d'état articulaire publié). L'odométrie réelle
-       vient de rf2o (recalage LiDAR), pas de la cinématique des roues. -->
+  <!-- Roues en joints fixes : pas d'encodeurs, pas de joint_states -->
   <xacro:macro name="wheel" params="prefix reflect">
     <link name="${prefix}_wheel_link">
       <visual>
         <origin xyz="0 0 0" rpy="${pi/2} 0 0"/>
-        <geometry>
-          <cylinder radius="${wheel_radius}" length="${wheel_width}"/>
-        </geometry>
+        <geometry><cylinder radius="${wheel_radius}" length="${wheel_width}"/></geometry>
         <material name="isimm_black"/>
       </visual>
       <collision>
         <origin xyz="0 0 0" rpy="${pi/2} 0 0"/>
-        <geometry>
-          <cylinder radius="${wheel_radius}" length="${wheel_width}"/>
-        </geometry>
+        <geometry><cylinder radius="${wheel_radius}" length="${wheel_width}"/></geometry>
       </collision>
       <xacro:cylinder_inertia mass="${wheel_mass}" r="${wheel_radius}" h="${wheel_width}"/>
@@ -116,5 +78,5 @@
       <parent link="base_link"/>
       <child link="${prefix}_wheel_link"/>
-      <origin xyz="${wheel_x} ${reflect * wheel_separation / 2.0} ${-base_link_z + wheel_z}" rpy="0 0 0"/>
+      <origin xyz="0 ${reflect * wheel_separation / 2.0} 0" rpy="0 0 0"/>
     </joint>
   </xacro:macro>
@@ -125,14 +87,10 @@
     <visual>
       <origin xyz="0 0 0" rpy="0 0 0"/>
-      <geometry>
-        <cylinder radius="${laser_radius}" length="${laser_length}"/>
-      </geometry>
+      <geometry><cylinder radius="${laser_radius}" length="${laser_length}"/></geometry>
       <material name="isimm_black"/>
     </visual>
     <collision>
       <origin xyz="0 0 0" rpy="0 0 0"/>
-      <geometry>
-        <cylinder radius="${laser_radius}" length="${laser_length}"/>
-      </geometry>
+      <geometry><cylinder radius="${laser_radius}" length="${laser_length}"/></geometry>
     </collision>
     <xacro:cylinder_inertia mass="0.2" r="${laser_radius}" h="${laser_length}"/>
@@ -141,5 +99,4 @@
     <parent link="base_link"/>
     <child link="laser_link"/>
-    <!-- laser_height est donné depuis base_footprint (sol) -> on retire base_link_z -->
     <origin xyz="${laser_x} ${laser_y} ${laser_height - base_link_z}" rpy="0 0 0"/>
   </joint>
@@ -148,14 +105,10 @@
     <visual>
       <origin xyz="0 0 0" rpy="0 0 0"/>
-      <geometry>
-        <box size="${imu_size} ${imu_size} ${imu_size}"/>
-      </geometry>
+      <geometry><box size="${imu_size} ${imu_size} ${imu_size}"/></geometry>
       <material name="isimm_red"/>
     </visual>
     <collision>
       <origin xyz="0 0 0" rpy="0 0 0"/>
-      <geometry>
-        <box size="${imu_size} ${imu_size} ${imu_size}"/>
-      </geometry>
+      <geometry><box size="${imu_size} ${imu_size} ${imu_size}"/></geometry>
     </collision>
     <xacro:box_inertia mass="0.05" x="${imu_size}" y="${imu_size}" z="${imu_size}"/>
@@ -164,5 +117,4 @@
     <parent link="base_link"/>
     <child link="imu_link"/>
-    <!-- imu_z est donné depuis base_footprint (sol) -> on retire base_link_z -->
     <origin xyz="${imu_x} ${imu_y} ${imu_z - base_link_z}" rpy="0 0 0"/>
   </joint>
